File: projects/FootSwitchBoard1/FootSwitchBoard1.brd (EAGLE design)
At the start: 50 x 50 mm, 46 parts

Commit message: Final version of files.
Connections:
- net GDUBINV: now also TC1044S.3
Routing:
- net N$1: track 21.5 -> 26.1 mm
- net N$113: track 2.54 -> 0.00 mm, vias 1 -> 0
- net N$112: track 2.54 -> 0.00 mm, vias 1 -> 0
- net GDUBINV: track 24.0 -> 21.6 mm, vias 0 -> 1
- net 9INDUBINV: track 33.4 -> 35.6 mm, vias 0 -> 1
- net N$6: track 24.5 -> 23.2 mm
- net N$11: track 12.6 -> 13.5 mm
