File: projects/DoubleClipperSwitchBoard/DoubleClipperSwitchBoard.brd (EAGLE design)
At the start: 18.2 x 16.9 mm, 12 parts

Commit message: Updated to use new clipper block.
Changed lines of the file:
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@@
 <contactref element="U$4" pad="P$2"/>
 <contactref element="U$5" pad="P$3"/>
-<contactref element="U$1" pad="P$2"/>
 <wire x1="4.064" y1="14.097" x2="1.524" y2="14.097" width="0.4064" layer="16"/>
 <wire x1="1.524" y1="14.097" x2="1.524" y2="11.557" width="0.4064" layer="16"/>
@@
 <wire x1="5.842" y1="13.081" x2="5.842" y2="12.065" width="0.4064" layer="1"/>
 <wire x1="5.842" y1="12.065" x2="6.096" y2="11.811" width="0.4064" layer="1"/>
-<wire x1="6.096" y1="11.811" x2="9.144" y2="11.811" width="0.4064" layer="1"/>
+<contactref element="U$1" pad="P$2"/>
+<wire x1="9.144" y1="11.811" x2="6.096" y2="11.811" width="0.4064" layer="1"/>
 </signal>
 <signal name="N$2">
